Commit message: Fixed tests using discrete collision manager in kdl_env_unit.cpp

File: tesseract_ros/test/urdf/pppbot.urdf (robot description, URDF)
Before this commit: robot pppbot, 5 links, 4 joints
Links:
- link obstacle1: geometry collision box size=.1 .1 .1; visual box size=.1 .1 .1
Joints:
- joint p2: limit lower=-.01 upper=.51 effort=10 velocity=1.0 -> lower=-.01 upper=.55 effort=10 velocity=1.0
